File: kicad/_autosave-LightSwitch.kicad_pcb (KiCad board)
At the start: 2 copper layers, 42 x 129.3 mm, 31 parts, among them J1 Screw_Terminal_01x02, J2 Conn_01x03_Male, Q1 MMBT2222A, SW1 SW_Push_LED, SW2 SW_Push_LED, SW3 SW_Push_LED, SW4 SW_Push_LED, SW5 SW_Push_LED, U1 LM2936-3.3, U2 SHT35-DIS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

Commit message: latect schematic
Parts:
- removed D3, D4: 1N4148WS, Diode_SMD:D_SOD-323
- removed R6: 27K, Resistor_SMD:R_0805_2012Metric
- removed R7: 2K, Resistor_SMD:R_0805_2012Metric
- added C6: 12pf, Capacitor_SMD:C_0805_2012Metric, F.Cu at (118.5, 93.2)
- added J3: Conn_ARM_JTAG_SWD_10, Connector_PinHeader_1.27mm:PinHeader_2x05_P1.27mm_Vertical_SMD, F.Cu at (117.6, 120.8)
- added J4: Conn_ARM_JTAG_SWD_10, Connector:Tag-Connect_TC2050-IDC-NL_2x05_P1.27mm_Vertical, F.Cu at (125.7, 120.7)
- added Q2: MMBT2222A, Package_TO_SOT_SMD:SOT-23, F.Cu at (115.2, 68.3)
- added REF**: MountingHole_3.2mm_M3, MountingHole:MountingHole_3.2mm_M3, F.Cu at (104.0, 84.0)
- added REF**: MountingHole_3.2mm_M3, MountingHole:MountingHole_3.2mm_M3, F.Cu at (138.0, 84.0)
- added REF**: MountingHole_3.2mm_M3, MountingHole:MountingHole_3.2mm_M3, F.Cu at (104.0, 44.0)
- added REF**: MountingHole_3.2mm_M3, MountingHole:MountingHole_3.2mm_M3, F.Cu at (104.0, 124.0)
- added REF**: MountingHole_3.2mm_M3, MountingHole:MountingHole_3.2mm_M3, F.Cu at (138.0, 44.0)
- added REF**: MountingHole_3.2mm_M3, MountingHole:MountingHole_3.2mm_M3, F.Cu at (138.0, 124.0)
- added U4: MX25R3235FM2xx0, Package_SO:SOP-8_5.28x5.23mm_P1.27mm, F.Cu at (116.1, 98.5)
- added Y1: 32.768kHz, Crystal:Crystal_SMD_3215-2Pin_3.2x1.5mm, F.Cu at (121.4, 91.9)
- C5: value 0.1u -> 12pf
- J1: moved to F.Cu
- J2: value Conn_01x03_Male -> Conn_01x06_Female; footprint Connector_PinHeader_2.54mm:PinHeader_1x03_P2.54mm_Vertical -> Connector_PinSocket_2.54mm:PinSocket_1x06_P2.54mm_Vertical
- R1: value 4.7K -> 2.2K
- R2: value 4.7K -> 10K
- R5: value 1K -> 10K
- SW1, SW2, SW3, SW4, SW5: moved to B.Cu
- U1: value LM2936-3.3 -> LM2936-3.0; footprint Package_TO_SOT_SMD:SOT-223 -> Package_TO_SOT_THT:TO-92_Inline
- U3: value ATtiny806-S -> E73-2G4M08S1C; footprint Package_SO:SOIC-20W_7.5x12.8mm_P1.27mm -> E73-2G4M08S1C:E73-2G4M08S1C
- moved R5 57.5 mm to (113.1, 105.5), turned to -90 degrees
- moved J1 50.6 mm to (118.4, 76.0)
- moved R1 39.0 mm to (115.2, 65.5), turned to 180 degrees
- moved J2 37.6 mm to (110.3, 117.7), turned to 180 degrees
- moved D2 24.2 mm to (125.7, 67.3), turned to 0 degrees
- moved U1 21.3 mm to (114.6, 90.9), turned to 180 degrees
- moved D1 18.3 mm to (115.0, 85.2)
- moved R4 18.1 mm to (119.0, 69.1), turned to 180 degrees
- moved Q1 17.4 mm to (119.1, 66.3)
- moved C2 16.4 mm to (112.3, 85.9), turned to 180 degrees
- moved C3 14.6 mm to (112.3, 87.9), turned to 0 degrees
- moved C1 13.7 mm to (112.3, 83.8), turned to 180 degrees
- moved R11 12.3 mm to (127.5, 84.5), turned to 180 degrees
- moved R9 11.6 mm to (126.8, 35.4)
- moved R10 11.6 mm to (126.8, 60.4)
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Connections:
- C5 pad 1: GND -> Net-(C5-Pad1)
- C5 pad 2: VDD -> GND
- J1 pad 1: /D1 -> /D2
- J1 pad 2: /D2 -> /D1
- J2 pad 1: VDD -> GND
- J2 pad 2: /PROG -> unconnected-(J2-Pad2)
- J2 pad 3: GND -> VDD
- R1 pad 1: VDD -> /DALI+
- R1 pad 2: /SDA -> Net-(Q2-Pad1)
- R2 pad 2: /SCL -> /SDA
- R5 pad 1: /DALI_TX -> VDD
- R5 pad 2: GND -> /SCL
- U3 pad 1: VDD -> /SW1
- U3 pad 10: /SDA -> unconnected-(U3-Pad10)
- U3 pad 11: /SCL -> Net-(C5-Pad1)
- U3 pad 12: /LED4 -> /CS
- U3 pad 13: /SW4 -> Net-(C6-Pad1)
- U3 pad 14: /LED5 -> /SIO_1
- U3 pad 15: /SW5 -> unconnected-(U3-Pad15)
- U3 pad 16: /PROG -> /SIO_2
- U3 pad 17: /TEMP_ALERT -> unconnected-(U3-Pad17)
- U3 pad 18: unconnected-(U3-Pad18) -> /SIO_3
- U3 pad 19: unconnected-(U3-Pad19) -> VDD
- U3 pad 2: /SW3 -> /LED1
- U3 pad 20: GND -> /SCLK
- U3 pad 3: /LED3 -> /SW2
- U3 pad 4: /DALI_TX -> /LED2
- U3 pad 5: /DALI_RX -> GND
- U3 pad 6: /SW2 -> /SW3
- U3 pad 7: /LED2 -> /LED3
- U3 pad 8: /SW1 -> /DALI_TX
- U3 pad 9: /LED1 -> /DALI_RX
Routing:
- net /~{RESET}: track 0.00 -> 54.3 mm, vias 0 -> 3
- net /SW2: track 0.00 -> 52.7 mm
- net /SWDCLK: track 0.00 -> 43.3 mm
- net /DALI_RX: track 65.1 -> 32.2 mm
- net /DALI_TX: track 64.6 -> 32.3 mm
- net /RX: track 0.00 -> 30.1 mm, vias 0 -> 1
- net /SWDIO: track 0.00 -> 27.7 mm, vias 0 -> 2
- net /TX: track 0.00 -> 26.6 mm, vias 0 -> 1
- net /LED2: track 5.52 -> 31.8 mm
- net /DALI+: track 7.44 -> 32.9 mm
- net VDD: track 124.3 -> 101.4 mm, vias 0 -> 2
- net /LED1: track 76.0 -> 57.8 mm
- net /SIO_1: track 0.00 -> 17.9 mm, vias 0 -> 2
- net /SIO_2: track 0.00 -> 17.9 mm, vias 0 -> 2
- net /CS: track 0.00 -> 17.9 mm, vias 0 -> 2
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- added copper zone on B.Cu, net GND
Other:
- board text added: "RX"
- board text added: "TX"
- board text removed: "PRG"
